File: PCB/3 Meter Dish LNA/002.35.20.15.20-001-PCB-LNA.kicad_pcb (KiCad board)
At the start: 2 copper layers, 86.4 x 49.4 mm, 29 parts, among them J1 Conn_Coaxial, J2 Conn_Coaxial, J3 Conn_Coaxial, U1 PMA2-63LN+, U2 PMA2-63LN+, U3 YAT-1A+, U4 L7805, U5 L7805

Commit message: Added document numbers
Other:
- board text added: "LNA footprint is also pin-compatible with: PMA2-123LN+ PMA2-153LN+"
Changed lines of the file:
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@@
     (effects (font (size 1.5 1.5) (thickness 0.3) bold) (justify left bottom))
+  )
+  (gr_text "LNA footprint is also pin-compatible with:\nPMA2-123LN+\nPMA2-153LN+" (at 177.8 167.005) (layer "Cmts.User")
+    (effects (font (size 1.5 1.5) (thickness 0.3) bold) (justify left top))
   )
   (segment (start 109.366 110.512) (end 115.0481 110.512) (width 0.63) (layer "F.Cu") (net 1))
