File: PCB/PMA3-14LN+/PMA3-14LN+.kicad_sch (KiCad schematic)
At the start: 19 parts, among them IC1 PMA3-14LN+, J1 Conn_Coaxial, J2 Conn_Coaxial, U1 L7806

Commit message: PMA3-14LN+ design complete sans signal launch tuning
Parts:
- L1, L2: footprint Inductor_SMD:L_0805_2012Metric -> Inductor_SMD:L_0402_1005Metric
- R1: footprint Resistor_SMD:R_0805_2012Metric -> Resistor_SMD:R_0402_1005Metric
Changed lines of the file:
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@@
       (effects (font (size 1.27 1.27)) (justify left))
     )
-    (property "Footprint" "Inductor_SMD:L_0805_2012Metric" (at 184.15 113.03 0)
+    (property "Footprint" "Inductor_SMD:L_0402_1005Metric" (at 184.15 113.03 0)
       (effects (font (size 1.27 1.27)) hide)
     )
@@
       (effects (font (size 1.27 1.27)) (justify left))
     )
-    (property "Footprint" "Inductor_SMD:L_0805_2012Metric" (at 107.95 113.03 0)
+    (property "Footprint" "Inductor_SMD:L_0402_1005Metric" (at 107.95 113.03 0)
       (effects (font (size 1.27 1.27)) hide)
     )
@@
       (effects (font (size 1.27 1.27)))
     )
-    (property "Footprint" "Resistor_SMD:R_0805_2012Metric" (at 132.08 88.9 0)
+    (property "Footprint" "Resistor_SMD:R_0402_1005Metric" (at 132.08 88.9 0)
       (effects (font (size 1.27 1.27)) hide)
     )

Commit message: Updated silkscreen and reference designators on EMS boards
Parts:
- renumbered IC1 to U1, U1 to U2
Changed lines of the file:
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@@
   (symbol (lib_id "Regulator_Linear:L7806") (at 143.51 45.72 0) (unit 1)
     (in_bom yes) (on_board yes) (dnp no) (fields_autoplaced)
-    (property "Reference" "U1" (at 143.51 39.37 0)
+    (property "Reference" "U2" (at 143.51 39.37 0)
       (effects (font (size 1.27 1.27)))
     )
@@
       (project "PMA3-14LN+"
         (path "/d268e3ca-8a18-4b0a-ac77-3cbf3521c83a"
-          (reference "U1") (unit 1)
+          (reference "U2") (unit 1)
         )
       )
@@
   (symbol (lib_id "PMA3-14LN+:PMA3-14LN+") (at 120.65 121.92 0) (unit 1)
     (in_bom yes) (on_board yes) (dnp no)
-    (property "Reference" "IC1" (at 173.99 115.4683 0)
+    (property "Reference" "U1" (at 173.99 115.4683 0)
       (effects (font (size 1.27 1.27)))
     )
@@
       (project "PMA3-14LN+"
         (path "/d268e3ca-8a18-4b0a-ac77-3cbf3521c83a"
-          (reference "IC1") (unit 1)
+          (reference "U1") (unit 1)
         )
       )
