File: PCB/PMA-183PLN+/PMA-183PLN+.kicad_sch (KiCad schematic)
At the start: 18 parts, among them J1 Conn_Coaxial, J2 Conn_Coaxial, U1 PMA-183PLN+, U2 MIC5219-2.6YM5-TR

Commit message: PMA-183PLN+ PCB Rev A completed
Parts:
- J1, J2: footprint footprints:SMA_Molex_73251-1153_EdgeMount_Horizontal_TunedOSH -> footprints:Mueller BU-1420761881
Changed lines of the file:
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@@
       (effects (font (size 1.27 1.27)) (justify left))
     )
-    (property "Footprint" "footprints:SMA_Molex_73251-1153_EdgeMount_Horizontal_TunedOSH" (at 81.28 124.46 0)
+    (property "Footprint" "footprints:Mueller BU-1420761881" (at 81.28 124.46 0)
       (effects (font (size 1.27 1.27)) hide)
     )
@@
       (effects (font (size 1.27 1.27)) (justify left))
     )
-    (property "Footprint" "footprints:SMA_Molex_73251-1153_EdgeMount_Horizontal_TunedOSH" (at 209.55 127 0)
-      (effects (font (size 1.27 1.27)) hide)
-    )
+    (property "Footprint" "footprints:Mueller BU-1420761881" (at 209.55 127 0)
+      (effects (font (size 1.27 1.27)) hide)
+    )
